File: hardware/kicad/zonnescherm.sch (KiCad schematic (older format))
At the start: 1 part

Commit message: Added documentation and Modex library
Parts:
- added K? (x4): FTR-LYCA, symbol FTR-LYCA
- added U?: ULN2003A, symbol ULN2003A
Connections:
- new net GND: U?.8 (GND)
Changed lines of the file:
@@
 LIBS:ESP8266
 LIBS:valves
+LIBS:modex
+LIBS:zonnescherm-cache
 EELAYER 25 0
 EELAYER END
@@
 	1    0    0    -1
 $EndComp
+$Comp
+L ULN2003A U?
+U 1 1 57851D26
+P 8250 3500
+F 0 "U?" H 8250 3600 50  0000 C CNN
+F 1 "ULN2003A" H 8250 3400 50  0000 C CNN
+F 2 "" H 8250 3500 50  0000 C CNN
+F 3 "" H 8250 3500 50  0000 C CNN
+	1    8250 3500
+	1    0    0    -1
+$EndComp
+$Comp
+L FTR-LYCA K?
+U 1 1 5785259B
+P 9950 1750
+F 0 "K?" H 9950 1900 50  0000 C CNN
+F 1 "FTR-LYCA" H 9950 1250 50  0000 C CNN
+F 2 "" H 9950 1750 50  0000 C CNN
+F 3 "" H 9950 1750 50  0000 C CNN
+	1    9950 1750
+	1    0    0    -1
+$EndComp
+$Comp
+L FTR-LYCA K?
+U 1 1 57852684
+P 9950 2550
+F 0 "K?" H 9950 2700 50  0000 C CNN
+F 1 "FTR-LYCA" H 9950 2050 50  0000 C CNN
+F 2 "" H 9950 2550 50  0000 C CNN
+F 3 "" H 9950 2550 50  0000 C CNN
+	1    9950 2550
+	1    0    0    -1
+$EndComp
+$Comp
+L FTR-LYCA K?
+U 1 1 5785271F
+P 10000 3350
+F 0 "K?" H 10000 3500 50  0000 C CNN
+F 1 "FTR-LYCA" H 10000 2850 50  0000 C CNN
+F 2 "" H 10000 3350 50  0000 C CNN
+F 3 "" H 10000 3350 50  0000 C CNN
+	1    10000 3350
+	1    0    0    -1
+$EndComp
+$Comp
+L FTR-LYCA K?
+U 1 1 5785279E
+P 10000 4200
+F 0 "K?" H 10000 4350 50  0000 C CNN
+F 1 "FTR-LYCA" H 10000 3700 50  0000 C CNN
+F 2 "" H 10000 4200 50  0000 C CNN
+F 3 "" H 10000 4200 50  0000 C CNN
+	1    10000 4200
+	1    0    0    -1
+$EndComp

Commit message: Added library symbols
Parts:
- added U?: LD1117S33TR, SOT-223, symbol LD1117S33TR
- added U?: IRM-05-5, symbol IRM-05-5
Changed lines of the file:
@@
+	1    0    0    -1
+$EndComp
+$Comp
+L LD1117S33TR U?
+U 1 1 57852872
+P 3000 1500
+F 0 "U?" H 3000 1750 50  0000 C CNN
+F 1 "LD1117S33TR" H 3000 1700 50  0000 C CNN
+F 2 "SOT-223" H 3000 1600 50  0000 C CNN
+F 3 "" H 3000 1500 50  0000 C CNN
+	1    3000 1500
+	1    0    0    -1
+$EndComp
+$Comp
+L IRM-05-5 U?
+U 1 1 57852A7E
+P 1700 1500
+F 0 "U?" H 1850 1304 50  0000 C CNN
+F 1 "IRM-05-5" H 1700 1700 50  0000 C CNN
+F 2 "" H 1700 1500 50  0000 C CNN
+F 3 "" H 1700 1500 50  0000 C CNN
+	1    1700 1500
 	1    0    0    -1
 $EndComp

Commit message: Added Python buienradar script
Parts:
- removed U?: LD1117S33TR, SOT-223, symbol LD1117S33TR
- added C? (x2): C, symbol C
- added C? (x2): CP, symbol CP
- added F?: 5A, symbol F_Small
- added P? (x3): CONN_01X04, symbol CONN_01X04
- added R? (x5): R, symbol R
- added SW? (x4): SW_PUSH, symbol SW_PUSH
- added U?: LM1117-3.3, symbol LM1117-3.3
Connections:
- net labels added: GND, N, P, P3V3, P5V
- wire segments 0 -> 18
Other:
- note added: "Mains"
- note added: "Sunshade 1"
- note added: "Sunshade 2"
- moved on the sheet: K?, U?

Commit message: Updated schematic
Parts:
- C? (x2): value C -> 100n
- P?: value CONN_01X04 -> CONN_MAINS
- P?: value CONN_01X04 -> CONN_SUNSHADE1
- P?: value CONN_01X04 -> CONN_SUNSHADE2
- R? (x5): value R -> 12k
- SW?: value SW_PUSH -> SW_UP_1
- SW?: value SW_PUSH -> SW_DOWN_1
- SW?: value SW_PUSH -> SW_UP_2
- SW?: value SW_PUSH -> SW_DOWN_2
- U?: symbol LM1117-3.3 -> LM1117-3.3-RESCUE-zonnescherm
Connections:
- net labels added: EN, GPIO0, GPIO15, GPIO2, PE, XRES
- wire segments 18 -> 96
Other:
- note removed: "Mains"
- note removed: "Sunshade 1"
- note removed: "Sunshade 2"
- moved on the sheet: C?, K?, P?, R?, SW?

Commit message: Added footprint library modex
Parts:
- added P1: ARDUINO-ISP, Pin_Headers:Pin_Header_Straight_1x06, symbol CONN_01X06
- added R1, R2: 12k, Resistors_SMD:R_0805_HandSoldering, symbol R
- C1: renamed from C?; value CP -> 100u/16V; footprint (none) -> Capacitors_SMD:c_elec_5x5.3
- C2, C3: renamed from C?; footprint (none) -> Capacitors_SMD:C_0805_HandSoldering
- C4: renamed from C?; value CP -> 10u/16V; footprint (none) -> Capacitors_SMD:c_elec_5x5.3
- F1: renamed from F?; value 5A -> 5AT
- K1: renamed from K?; value FTR-LYCA -> K1-ON/OFF
- K2: renamed from K?; value FTR-LYCA -> K1-UP/DOWN
- K3: renamed from K?; value FTR-LYCA -> K2-ON/OFF
- K4: renamed from K?; value FTR-LYCA -> K2-UP/DOWN
- R3, R4, R5, R6, R7: renamed from R?; footprint (none) -> Resistors_SMD:R_0805_HandSoldering
- SW1, SW2, SW3, SW4: renamed from SW?; footprint (none) -> Buttons_Switches_ThroughHole:SW_PUSH_SMALL
- U2: renamed from U?; footprint (none) -> TO_SOT_Packages_SMD:TO-263-3Lead
- U3: renamed from U?; footprint (none) -> ESP8266:ESP-12E
- U4: renamed from U?; footprint (none) -> SMD_Packages:SO-16-N
- gave numbers to parts that had none: 4
Connections:
- net labels added: GPIO4, GPIO5, RXD, TXD
- wire segments 96 -> 123
Other:
- moved on the sheet: F1, P2, P3, P4, SW1, SW2, SW3, SW4, U4

Commit message: Added new footprint
Parts:
- F1: footprint (none) -> Fuse_Holders_and_Fuses:Fuseholder5x20_horiz_SemiClosed_Casing10x25mm
- K1, K2, K3, K4: footprint (none) -> modex:FTR_LY
Changed lines of the file:
@@
 F 0 "K1" H 8600 2250 50  0000 C CNN
 F 1 "K1-ON/OFF" H 8600 1600 50  0000 C CNN
-F 2 "" H 8600 2100 50  0001 C CNN
+F 2 "modex:FTR_LY" H 8600 2100 50  0001 C CNN
 F 3 "" H 8600 2100 50  0000 C CNN
 	1    8600 2100
@@
 F 0 "K2" H 8600 3050 50  0000 C CNN
 F 1 "K1-UP/DOWN" H 8600 2400 50  0000 C CNN
-F 2 "" H 8600 2900 50  0001 C CNN
+F 2 "modex:FTR_LY" H 8600 2900 50  0001 C CNN
 F 3 "" H 8600 2900 50  0000 C CNN
 	1    8600 2900
@@
 F 0 "K3" H 8600 3850 50  0000 C CNN
 F 1 "K2-ON/OFF" H 8600 3200 50  0000 C CNN
-F 2 "" H 8600 3700 50  0001 C CNN
+F 2 "modex:FTR_LY" H 8600 3700 50  0001 C CNN
 F 3 "" H 8600 3700 50  0000 C CNN
 	1    8600 3700
@@
 F 0 "K4" H 8600 4700 50  0000 C CNN
 F 1 "K2-UP/DOWN" H 8600 4050 50  0000 C CNN
-F 2 "" H 8600 4550 50  0001 C CNN
+F 2 "modex:FTR_LY" H 8600 4550 50  0001 C CNN
 F 3 "" H 8600 4550 50  0000 C CNN
 	1    8600 4550
@@
 F 0 "F1" H 9960 1960 50  0000 L CNN
 F 1 "5AT" H 9880 1840 50  0000 L CNN
-F 2 "" H 10000 1900 50  0001 C CNN
+F 2 "Fuse_Holders_and_Fuses:Fuseholder5x20_horiz_SemiClosed_Casing10x25mm" H 10000 1900 50  0001 C CNN
 F 3 "" H 10000 1900 50  0000 C CNN
 	1    10000 1900

Commit message: Added footprints
Parts:
- U1: footprint (none) -> modex:IRM-05
Changed lines of the file:
@@
 F 0 "U1" H 2850 1354 50  0000 C CNN
 F 1 "IRM-05-5" H 2700 1750 50  0000 C CNN
-F 2 "" H 2700 1550 50  0001 C CNN
+F 2 "modex:IRM-05" H 2700 1550 50  0001 C CNN
 F 3 "" H 2700 1550 50  0000 C CNN
 	1    2700 1550

Commit message: Added AKL-330-4 footprint
Parts:
- P2, P3, P4: footprint (none) -> modex:AKL-330-4
Changed lines of the file:
@@
 F 0 "P2" H 10550 2300 50  0000 C CNN
 F 1 "CONN_MAINS" V 10650 2050 50  0000 C CNN
-F 2 "" H 10550 2050 50  0001 C CNN
+F 2 "modex:AKL-330-4" H 10550 2050 50  0001 C CNN
 F 3 "" H 10550 2050 50  0000 C CNN
 	1    10550 2050
@@
 F 0 "P3" H 10550 3250 50  0000 C CNN
 F 1 "CONN_SUNSHADE1" V 10650 3000 50  0000 C CNN
-F 2 "" H 10550 3000 50  0001 C CNN
+F 2 "modex:AKL-330-4" H 10550 3000 50  0001 C CNN
 F 3 "" H 10550 3000 50  0000 C CNN
 	1    10550 3000
@@
 F 0 "P4" H 10550 4900 50  0000 C CNN
 F 1 "CONN_SUNSHADE2" V 10650 4650 50  0000 C CNN
-F 2 "" H 10550 4650 50  0001 C CNN
+F 2 "modex:AKL-330-4" H 10550 4650 50  0001 C CNN
 F 3 "" H 10550 4650 50  0000 C CNN
 	1    10550 4650
